File: EagleFiles/YouHaveBeenBlinded.brd (EAGLE design)
At the start: 101.6 x 101.6 mm, 13 parts, among them J1 5.5x2.1mm Barrel

Commit message: Final release of Eagle and Gerber files
Connections:
- net +3V: now also J1.VIN0; no longer J1.GND, J1.P$4
- net GND: now also J1.P$4
Routing:
- net +3V: track 131.4 -> 149.1 mm
Changed lines of the file:
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@@
 </polygon>
 <contactref element="MOTOR-" pad="MP"/>
+<contactref element="J1" pad="P$4"/>
 </signal>
 <signal name="+3V">
@@
 <contactref element="SW2" pad="1"/>
 <contactref element="SW1" pad="1"/>
-<contactref element="J1" pad="P$4"/>
-<contactref element="J1" pad="GND"/>
 <wire x1="83.5406" y1="19.7612" x2="84.2518" y2="19.7612" width="0.6096" layer="1"/>
-<wire x1="56.5" y1="81.28" x2="56.5" y2="75.18" width="0.6096" layer="16"/>
 <wire x1="50.8" y1="19.05" x2="46.99" y2="22.86" width="1.016" layer="1"/>
 <wire x1="59.69" y1="19.05" x2="50.8" y2="19.05" width="1.016" layer="1"/>
@@
 <wire x1="86.36" y1="26.67" x2="86.36" y2="36.83" width="1.016" layer="1"/>
 <wire x1="83.82" y1="39.37" x2="83.5406" y2="40.0812" width="1.016" layer="1"/>
-<wire x1="83.82" y1="55.88" x2="64.77" y2="74.93" width="1.016" layer="16"/>
-<wire x1="64.77" y1="74.93" x2="57.15" y2="74.93" width="1.016" layer="16"/>
-<wire x1="83.82" y1="40.64" x2="83.82" y2="55.88" width="1.016" layer="16"/>
-<wire x1="57.15" y1="74.93" x2="56.5" y2="75.18" width="1.016" layer="16"/>
 <wire x1="83.82" y1="40.64" x2="83.5406" y2="40.0812" width="1.016" layer="16"/>
 <wire x1="73.66" y1="26.67" x2="72.39" y2="27.94" width="1.016" layer="1"/>
 <wire x1="86.36" y1="26.67" x2="73.66" y2="26.67" width="1.016" layer="1"/>
+<contactref element="J1" pad="VIN0"/>
+<wire x1="45.1" y1="81.28" x2="45.72" y2="81.28" width="0.4064" layer="16"/>
+<wire x1="45.72" y1="81.28" x2="45.72" y2="85.09" width="1.016" layer="16"/>
+<wire x1="45.72" y1="85.09" x2="62.23" y2="85.09" width="1.016" layer="16"/>
+<wire x1="62.23" y1="85.09" x2="83.82" y2="63.5" width="1.016" layer="16"/>
+<wire x1="83.82" y1="63.5" x2="83.82" y2="40.64" width="1.016" layer="16"/>
 </signal>
 <signal name="N$4">
